File: hardware/design/get-smart-controller.kicad_sch (KiCad schematic)
At the start: 17 parts, among them J1 USB_B_Micro, J2 BOOT, J3 UART, U1 ESP32-S3-WROOM-1, U2 AMS1117-3.3, U3 Ai-Thinker-Ra-02

Commit message: Updated PCB with holes
Parts:
- D1: value 1N5819 -> SS14; footprint Diode_SMD:D_0805_2012Metric_Pad1.15x1.40mm_HandSolder -> Diode_SMD:D_SOD-323_HandSoldering
Changed lines of the file:
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@@
 			)
 		)
-		(property "Value" "1N5819"
+		(property "Value" "SS14"
 			(at 60.0075 148.59 0)
 			(effects
@@
 			)
 		)
-		(property "Footprint" "Diode_SMD:D_0805_2012Metric_Pad1.15x1.40mm_HandSolder"
+		(property "Footprint" "Diode_SMD:D_SOD-323_HandSoldering"
 			(at 59.69 147.955 0)
 			(effects

Commit message: Added RGB led, and fixed foorptint for USB Micro
Parts:
- removed J2: BOOT, Connector_PinHeader_2.54mm:PinHeader_1x02_P2.54mm_Vertical, symbol Connector:Conn_01x02_Pin
- added D2: SK6812, LED_SMD:LED_SK6812_PLCC4_5.0x5.0mm_P3.2mm, symbol LED:SK6812
- added Q1: MMBT3904, Package_TO_SOT_SMD:SOT-23, symbol Transistor_BJT:MMBT3904
- added R3, R4: 1k, Resistor_SMD:R_0805_2012Metric_Pad1.20x1.40mm_HandSolder, symbol Device:R
- J1: footprint Connector_USB:USB_Micro-B_Wuerth_629105150521 -> Connector_USB:USB_Micro-B_Custom
- J3: footprint Connector_PinHeader_2.54mm:PinHeader_1x04_P2.54mm_Vertical -> Connector_JST:JST_PH_S4B-PH-K_1x04_P2.00mm_Horizontal; symbol Connector:Conn_01x04_Pin -> Connector:Conn_01x04_Socket
Connections:
- net +3V3: now also J3.1 (Pin_1); no longer J3.4 (Pin_4)
- net +5V: now also D2.3 (VDD), R3.1
- net GND: now also J3.4 (Pin_4), D2.1 (VSS), Q1.2 (E); no longer J3.1 (Pin_1)
- net RX: now also J3.2 (Pin_2); no longer J3.3 (Pin_3)
- net TX: now also J3.3 (Pin_3); no longer J3.2 (Pin_2)
- net RGB: now reaches U1.29 (SPIIO7/GPIO36/FSPICLK/SUBSPICLK)
- net RGB: now also R4.1
- new net: Q1.3 (C), R3.2
- new net: Q1.1 (B), R4.2
- no-connect marks 26 -> 25
Other:
- moved on the sheet: C7, R1, R2, U3
